Commit message: Adding files for the hardware interface. It builds, and sim can be run by setting the sim_mode to true, but it is currently untested with the hardware.

File: src/midas_moveit_config/config/midas.ros2_control.xacro (robot description, xacro)
@@ -2,51 +2,105 @@
 <robot xmlns:xacro="http://www.ros.org/wiki/xacro">
     <xacro:macro name="midas_ros2_control" params="name initial_positions_file">
-        <xacro:property name="initial_positions" value="${load_yaml(initial_positions_file)['initial_positions']}"/>
-        <ros2_control name="${name}" type="system">
-            <hardware>
-                <!-- By default, set up controllers for simulation. This won't work on real hardware -->
-                <plugin>mock_components/GenericSystem</plugin>
-            </hardware>
-            <joint name="J1">
-                <command_interface name="position"/>
-                <state_interface name="position">
-                  <param name="initial_value">${initial_positions['J1']}</param>
-                </state_interface>
-                <state_interface name="velocity"/>
-                <state_interface name="effort"/>
-            </joint>
-            <joint name="J2">
-                <command_interface name="position"/>
-                <state_interface name="position">
-                  <param name="initial_value">${initial_positions['J2']}</param>
-                </state_interface>
-                <state_interface name="velocity"/>
-                <state_interface name="effort"/>
-            </joint>
-            <joint name="J3">
-                <command_interface name="position"/>
-                <state_interface name="position">
-                  <param name="initial_value">${initial_positions['J3']}</param>
-                </state_interface>
-                <state_interface name="velocity"/>
-                <state_interface name="effort"/>
-            </joint>
-            <joint name="J4">
-                <command_interface name="position"/>
-                <state_interface name="position">
-                  <param name="initial_value">${initial_positions['J4']}</param>
-                </state_interface>
-                <state_interface name="velocity"/>
-                <state_interface name="effort"/>
-            </joint>
-            <joint name="J5">
-                <command_interface name="position"/>
-                <state_interface name="position">
-                  <param name="initial_value">${initial_positions['J5']}</param>
-                </state_interface>
-                <state_interface name="velocity"/>
-                <state_interface name="effort"/>
-            </joint>
-        </ros2_control>
+        <xacro:if value="$(arg sim_mode)">
+            <xacro:property name="initial_positions" value="${load_yaml(initial_positions_file)['initial_positions']}"/>
+            <ros2_control name="sim_robot" type="system">
+                <hardware>
+                    <!-- By default, set up controllers for simulation. This won't work on real hardware -->
+                    <plugin>mock_components/GenericSystem</plugin>
+                </hardware>
+                <joint name="J1">
+                    <command_interface name="position"/>
+                    <state_interface name="position">
+                      <param name="initial_value">${initial_positions['J1']}</param>
+                    </state_interface>
+                    <state_interface name="velocity"/>
+                    <state_interface name="effort"/>
+                </joint>
+                <joint name="J2">
+                    <command_interface name="position"/>
+                    <state_interface name="position">
+                      <param name="initial_value">${initial_positions['J2']}</param>
+                    </state_interface>
+                    <state_interface name="velocity"/>
+                    <state_interface name="effort"/>
+                </joint>
+                <joint name="J3">
+                    <command_interface name="position"/>
+                    <state_interface name="position">
+                      <param name="initial_value">${initial_positions['J3']}</param>
+                    </state_interface>
+                    <state_interface name="velocity"/>
+                    <state_interface name="effort"/>
+                </joint>
+                <joint name="J4">
+                    <command_interface name="position"/>
+                    <state_interface name="position">
+                      <param name="initial_value">${initial_positions['J4']}</param>
+                    </state_interface>
+                    <state_interface name="velocity"/>
+                    <state_interface name="effort"/>
+                </joint>
+                <joint name="J5">
+                    <command_interface name="position"/>
+                    <state_interface name="position">
+                      <param name="initial_value">${initial_positions['J5']}</param>
+                    </state_interface>
+                    <state_interface name="velocity"/>
+                    <state_interface name="effort"/>
+                </joint>
+            </ros2_control>
+        </xacro:if>
+        <xacro:unless value="$(arg sim_mode)">
+            <ros2_control name="real_robot" type="system">
+                <hardware>
+                    <plugin>midas_interface/MidasInterface</plugin>
+                    <param name="J1">J1</param>
+                    <param name="J2">J2</param>
+                    <param name="J3">J3</param>
+                    <param name="J4">J4</param>
+                    <param name="J5">J5</param>
+                </hardware>
+                <joint name="J1">
+                    <command_interface name="position">
+                        <param name="min">-360</param>
+                        <param name="max">360</param>
+                    </command_interface>
+                    <state_interface name="position"/>
+                    <state_interface name="velocity"/>
+                </joint>
+                <joint name="J2">
+                    <command_interface name="position">
+                        <param name="min">-360</param>
+                        <param name="max">360</param>
+                    </command_interface>
+                    <state_interface name="position"/>
+                    <state_interface name="velocity"/>
+                </joint>
+                <joint name="J3">
+                    <command_interface name="position">
+                        <param name="min">-360</param>
+                        <param name="max">360</param>
+                    </command_interface>
+                    <state_interface name="position"/>
+                    <state_interface name="velocity"/>
+                </joint>
+                <joint name="J4">
+                    <command_interface name="position">
+                        <param name="min">-360</param>
+                        <param name="max">360</param>
+                    </command_interface>
+                    <state_interface name="position"/>
+                    <state_interface name="velocity"/>
+                </joint>
+                <joint name="J5">
+                    <command_interface name="position">
+                        <param name="min">-360</param>
+                        <param name="max">360</param>
+                    </command_interface>
+                    <state_interface name="position"/>
+                    <state_interface name="velocity"/>
+                </joint>
+            </ros2_control>
+        </xacro:unless>
     </xacro:macro>
 </robot>

File: src/midas_moveit_config/config/midas.urdf.xacro (robot description, xacro)
@@ -2,4 +2,5 @@
 <robot xmlns:xacro="http://www.ros.org/wiki/xacro" name="midas">
     <xacro:arg name="initial_positions_file" default="initial_positions.yaml" />
+    <xacro:arg name="sim_mode" default="false"/>
     <!-- Import midas urdf file -->
     <xacro:include filename="$(find robot_description)/urdf/robot.urdf" />

Commit message: robot spawns in gazebo. Error when motion planning

File: src/midas_moveit_config/config/midas.ros2_control.xacro (robot description, xacro)
@@ -2,9 +2,9 @@
 <robot xmlns:xacro="http://www.ros.org/wiki/xacro">
     <xacro:macro name="midas_ros2_control" params="name initial_positions_file">
-        <xacro:property name="initial_positions" value="${load_yaml(initial_positions_file)['initial_positions']}"/>
+        <xacro:property name="initial_positions" value="${xacro.load_yaml(initial_positions_file)['initial_positions']}"/>
         <ros2_control name="${name}" type="system">
             <hardware>
                 <!-- By default, set up controllers for simulation. This won't work on real hardware -->
-                <plugin>mock_components/GenericSystem</plugin>
+                <plugin>ign_ros2_control/IgnitionSystem</plugin>
             </hardware>
             <joint name="J1">

File: src/midas_moveit_config/config/midas.urdf.xacro (robot description, xacro)
@@ -3,7 +3,13 @@
     <xacro:arg name="initial_positions_file" default="initial_positions.yaml" />
     <!-- Import midas urdf file -->
-    <xacro:include filename="$(find robot_description)/urdf/robot.urdf" />
+    <xacro:include filename="$(find robot_description)/urdf_no_eff/robot.urdf" />
     <!-- Import control_xacro -->
     <xacro:include filename="midas.ros2_control.xacro" />
     <xacro:midas_ros2_control name="FakeSystem" initial_positions_file="$(arg initial_positions_file)"/>
+    <gazebo>
+        <plugin name="ign_ros2_control::IgnitionROS2ControlPlugin" filename="libign_ros2_control-system.so">
+        <!-- Optional configuration (e.g., control period) -->
+        <parameters>$(find midas_moveit_config)/config/ros2_controllers.yaml</parameters>
+        </plugin>
+    </gazebo>
 </robot>
