Commit message: - modified urdf to use new name format

File: src/robot_description/urdf/robot.urdf (robot description, URDF)
Before this commit: robot midas, 6 links, 5 joints
Links:
- removed link base_link
- added link base, mass 1.7134; collision mesh filename=package://robot_description/urdf/assets/bottom_cover.stl; collision mesh filename=package://robot_description/urdf/assets/carrier.stl
- link j2: geometry collision mesh filename=package://robot_description/urdf/assets/bottom_cover.stl; collision mesh filename=package://robot_description/urdf/assets/carrier.stl
- link j3: geometry collision mesh filename=package://robot_description/urdf/assets/m_17_motor_mount.stl; collision mesh filename=package://robot_description/urdf/assets/m_17he19_2004s.stl
- link j4: geometry collision mesh filename=package://robot_description/urdf/assets/horizontal_mount_17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; collision mesh filename=package://robot_description/urdf/assets/m_17hs08_1004s.stl
- link j5: geometry collision mesh filename=package://robot_description/urdf/assets/j6_mount.stl; collision mesh filename=package://robot_description/urdf/assets/m_17hs08_1004s.stl
- link platform: geometry collision mesh filename=package://robot_description/urdf/assets/composite_part_1__2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; collision mesh filename=package://robot_description/urdf/assets/flange2.stl
Joints:
- joint J1: limit lower=-6.28319 upper=6.28319 effort=10 velocity=10 -> lower=-2.28464 upper=3.99854 effort=1.85 velocity=10; origin xyz=4.36341e-18 -4.06324e-18 0.017 rpy=-3.14159 1.54087e-16 -0.10863 -> xyz=2.90478e-18 2.51725e-17 0.017 rpy=-3.14159 7.29843e-17 2.27611; parent base_link -> base
- joint J2: limit lower=-6.28319 upper=6.28319 effort=10 velocity=10 -> lower=0 upper=6.28319 effort=24.8 velocity=10; origin xyz=-2.20347e-16 0.108596 -0.03657 rpy=1.5708 -1.5708 0 -> xyz=-0.0820821 -0.071103 -0.03657 rpy=-2.42774 -1.5708 0
- joint J3: limit lower=-6.28319 upper=6.28319 effort=10 velocity=10 -> lower=-6.28319 upper=3.71518e-10 effort=7.4 velocity=10; origin xyz=-0.1906 -9.39422e-18 0.0381 rpy=-3.14159 -2.63382e-15 -1.3964e-09 -> xyz=-0.1906 -4.91006e-17 0.0381 rpy=-3.14159 -2.08945e-15 -1.3964e-09
- joint J4: limit lower=-6.28319 upper=6.28319 effort=10 velocity=10 -> lower=-4.7123 upper=1.57088 effort=0.55 velocity=10; origin xyz=-8.88178e-16 0.0339458 -0.026 rpy=1.5708 0.000106634 -3.14159 -> xyz=-8.32667e-16 0.0339458 -0.026 rpy=1.5708 8.51991e-05 -3.14159
- joint J5: limit lower=-6.28319 upper=6.28319 effort=10 velocity=10 -> lower=-3.99854 upper=2.28464 effort=0.16 velocity=10; origin xyz=0.02925 -1.56819e-15 0.22388 rpy=1.5708 0.00822554 -1.5708 -> xyz=0.02925 -1.31145e-15 0.22388 rpy=1.5708 0.713848 -1.5708

Commit message: simplified URDF model for easier manipulation and less computational load

File: src/robot_description/urdf/robot.urdf (robot description, URDF)
Before this commit: robot midas, 6 links, 5 joints
Links:
- removed link platform
- added link j1, mass 2.59; collision mesh filename=package://robot_description/urdf/assets/j1.stl; visual mesh filename=package://robot_description/urdf/assets/j1.stl
- link base: mass 1.7134 -> 8; geometry collision mesh filename=package://robot_description/urdf/assets/base.stl; visual mesh filename=package://robot_description/urdf/assets/base.stl
- link j2: mass 1.74979 -> 1.75; geometry collision mesh filename=package://robot_description/urdf/assets/j2.stl; visual mesh filename=package://robot_description/urdf/assets/j2.stl
- link j3: mass 0.472139 -> 0.472; geometry collision mesh filename=package://robot_description/urdf/assets/j3.stl; visual mesh filename=package://robot_description/urdf/assets/j3.stl
- link j4: mass 0.349009 -> 0.349; geometry collision mesh filename=package://robot_description/urdf/assets/j4.stl; visual mesh filename=package://robot_description/urdf/assets/j4.stl
- link j5: mass 0.217895 -> 0.218; geometry collision mesh filename=package://robot_description/urdf/assets/j5.stl; visual mesh filename=package://robot_description/urdf/assets/j5.stl
Joints:
- removed joint J1
- removed joint J2
- removed joint J3
- removed joint J4
- removed joint J5
- added joint j1: type revolute, parent base, child j1, origin xyz=0.323698 -0.00379571 0.0109293 rpy=0 -0 -0.239754, axis 0 0 1, limit lower=-3.141592653589793 upper=3.141592653589793 effort=10 velocity=10
- added joint j2: type revolute, parent j1, child j2, origin xyz=0.085 5.55112e-17 -0.03632 rpy=1.5708 0.934222 -1.5708, axis 0 0 1, limit lower=-3.141592653589793 upper=3.141592653589793 effort=10 velocity=10
- added joint j3: type revolute, parent j2, child j3, origin xyz=0.1956 4.16334e-17 0 rpy=-3.14159 -8.24569e-17 -1.9746, axis 0 0 1, limit lower=-3.141592653589793 upper=3.141592653589793 effort=10 velocity=10
- added joint j4: type revolute, parent j3, child j4, origin xyz=0.0432636 0 -0.0643 rpy=-1.5708 -1.90593e-19 -1.5708, axis 0 0 1, limit lower=-3.141592653589793 upper=3.141592653589793 effort=10 velocity=10
- added joint j5: type revolute, parent j4, child j5, origin xyz=0.00083682 0.0150466 0.241638 rpy=-1.5708 0.00650835 3.08603, axis 0 0 1, limit lower=-3.141592653589793 upper=3.141592653589793 effort=10 velocity=10

Commit message: corrected launch file to use sdf format for launching robot switched to ign-gazebo for simulation
steps to recreate:
	sudo apt-get install ros-humble-ros-gz
	sudo apt-get install ros-humble-ros-ign-bridge

	colcon build
	source install/setup.bash
	ros2 launch robot_description gazebo_launch.py

there may be an issue with environment variable pathing:
run the following in terminal, delete build dir, delete install dir:
	unset AMENT_PREFIX_PATH
	unset CMAKE_PREFIX_PATH
	unset COLCON_PREFIX_PATH
	unset LD_LIBRARY_PATH
	unset PYTHONPATH
colcon build and source install directory

known issues:
	robot spawns upside down

File: src/robot_description/urdf/robot.urdf (robot description, URDF)
Before this commit: robot midas, 6 links, 5 joints
Links:
- removed link j1
- removed link j2
- removed link j3
- removed link j4
- removed link j5
- added link link_j1, mass 2.59; collision mesh filename=package://robot_description/urdf/assets/link_j1.stl; visual mesh filename=package://robot_description/urdf/assets/link_j1.stl
- added link link_j2, mass 1.75; collision mesh filename=package://robot_description/urdf/assets/link_j2.stl; visual mesh filename=package://robot_description/urdf/assets/link_j2.stl
- added link link_j3, mass 0.472; collision mesh filename=package://robot_description/urdf/assets/link_j3.stl; visual mesh filename=package://robot_description/urdf/assets/link_j3.stl
- added link link_j4, mass 0.349; collision mesh filename=package://robot_description/urdf/assets/link_j4.stl; visual mesh filename=package://robot_description/urdf/assets/link_j4.stl
- added link link_j5, mass 0.218; collision mesh filename=package://robot_description/urdf/assets/link_j5.stl; visual mesh filename=package://robot_description/urdf/assets/link_j5.stl
Joints:
- joint j1: child j1 -> link_j1
- joint j2: child j2 -> link_j2; parent j1 -> link_j1
- joint j3: child j3 -> link_j3; parent j2 -> link_j2
- joint j4: child j4 -> link_j4; parent j3 -> link_j3
- joint j5: child j5 -> link_j5; parent j4 -> link_j4

Commit message: adding rest of files that needed to be in last commit

File: src/robot_description/urdf/robot.urdf (robot description, URDF)
Before this commit: robot midas, 6 links, 5 joints
Joints:
- joint j1: origin xyz=0.323698 -0.00379571 0.0109293 rpy=0 -0 -0.239754 -> xyz=-9.50428e-19 0.0585 0.1036 rpy=3.14159 -0 1.5708
- joint j2: origin xyz=0.085 5.55112e-17 -0.03632 rpy=1.5708 0.934222 -1.5708 -> xyz=0.086 2.23158e-19 -0.03632 rpy=-3.14159 1.5708 0
- joint j3: origin xyz=0.1956 4.16334e-17 0 rpy=-3.14159 -8.24569e-17 -1.9746 -> xyz=0.2086 1.27555e-17 0.001 rpy=-3.14159 1.11022e-15 -1.5708
- joint j4: origin xyz=0.0432636 0 -0.0643 rpy=-1.5708 -1.90593e-19 -1.5708 -> xyz=0.0432651 0 -0.0643 rpy=-1.5708 -3.69779e-32 -1.5708
- joint j5: origin xyz=0.00083682 0.0150466 0.241638 rpy=-1.5708 0.00650835 3.08603 -> xyz=1.11022e-16 0.0160737 0.242638 rpy=-1.5708 -1.66533e-15 3.14159

Commit message: enabled gazebo simulation to recieve messages from moveit 2 main issue lied within the robot.urdf file. was missing:
<gazebo>

  <plugin filename="libgazebo_ros2_control.so" name="gazebo_ros2_control">

    <parameters>$(find simple_moveit)/config/ros2_controllers.yaml</parameters>

   </plugin>

</gazebo>

reason being that although we were using the gazebo_ros2_control plugin within the robot_description.urdf.xacro, we never defined what it was

File: src/robot_description/urdf/robot.urdf (robot description, URDF)
Before this commit: robot robot_description, 6 links, 5 joints
Links:
- added link world
Joints:
- added joint world_to_base: type fixed, parent world, child base, origin xyz=0 0 0 rpy=0 0 0

File: src/simple_moveit/config/robot_description.ros2_control.xacro (robot description, xacro)
@@ -6,5 +6,5 @@
             <hardware>
                 <!-- By default, set up controllers for simulation. This won't work on real hardware -->
-                <plugin>mock_components/GenericSystem</plugin>
+        <plugin>gazebo_ros2_control/GazeboSystem</plugin>
             </hardware>
             <joint name="j1">

Commit message: added tags to allow for effor to be read out

File: src/robot_description/urdf/robot.urdf (robot description, URDF)
Before this commit: robot robot_description, 7 links, 6 joints
Links:
- removed link world
- added link payload, mass 2.0
Joints:
- removed joint world_to_base
- added joint payload_joint: type fixed, parent link_j5, child payload
- joint j1: limit lower=-3.141592653589793 upper=3.141592653589793 effort=10 velocity=10 -> lower=-3.141592653589793 upper=3.141592653589793 effort=1.85 velocity=10
- joint j2: limit lower=-3.141592653589793 upper=3.141592653589793 effort=10 velocity=10 -> lower=-3.141592653589793 upper=3.141592653589793 effort=24.8 velocity=10
- joint j3: limit lower=-3.141592653589793 upper=3.141592653589793 effort=10 velocity=10 -> lower=-3.141592653589793 upper=3.141592653589793 effort=7.4 velocity=10
- joint j4: limit lower=-3.141592653589793 upper=3.141592653589793 effort=10 velocity=10 -> lower=-3.141592653589793 upper=3.141592653589793 effort=0.55 velocity=10
- joint j5: limit lower=-3.141592653589793 upper=3.141592653589793 effort=10 velocity=10 -> lower=-3.141592653589793 upper=3.141592653589793 effort=0.16 velocity=10

File: src/simple_moveit/config/robot_description.ros2_control.xacro (robot description, xacro)
@@ -6,14 +6,26 @@
             <hardware>
                 <!-- By default, set up controllers for simulation. This won't work on real hardware -->
-        <plugin>gazebo_ros2_control/GazeboSystem</plugin>
+              <plugin>gazebo_ros2_control/GazeboSystem</plugin>
+              <!-- These params force effort interface activation -->
+              <param name="robot_sim_type">gazebo_sim</param>
+              <param name="use_sim_time">true</param>
             </hardware>
             <joint name="j1">
+                <dynamics>
+                  <damping>0.1</damping>  <!-- Friction value (0.1-1.0 is reasonable) -->
+                  <friction>0.5</friction>  <!-- Static friction -->
+                </dynamics>
                 <command_interface name="position"/>
                 <state_interface name="position">
                   <param name="initial_value">${initial_positions['j1']}</param>
                 </state_interface>
-                <state_interface name="velocity"/>
+              <state_interface name="velocity"/>
+              <state_interface name="effort"/>
             </joint>
             <joint name="j2">
+                <dynamics>
+                  <damping>0.1</damping>  <!-- Friction value (0.1-1.0 is reasonable) -->
+                  <friction>0.5</friction>  <!-- Static friction -->
+                </dynamics>
                 <command_interface name="position"/>
                 <state_interface name="position">
@@ -21,6 +33,11 @@
                 </state_interface>
                 <state_interface name="velocity"/>
+                <state_interface name="effort"/>
             </joint>
             <joint name="j3">
+                <dynamics>
+                  <damping>0.1</damping>  <!-- Friction value (0.1-1.0 is reasonable) -->
+                  <friction>0.5</friction>  <!-- Static friction -->
+                </dynamics>
                 <command_interface name="position"/>
                 <state_interface name="position">
@@ -28,6 +45,11 @@
                 </state_interface>
                 <state_interface name="velocity"/>
+                <state_interface name="effort"/>
             </joint>
             <joint name="j4">
+                <dynamics>
+                  <damping>0.1</damping>  <!-- Friction value (0.1-1.0 is reasonable) -->
+                  <friction>0.5</friction>  <!-- Static friction -->
+                </dynamics>
                 <command_interface name="position"/>
                 <state_interface name="position">
@@ -35,6 +57,11 @@
                 </state_interface>
                 <state_interface name="velocity"/>
+                <state_interface name="effort"/>
             </joint>
             <joint name="j5">
+                <dynamics>
+                  <damping>0.1</damping>  <!-- Friction value (0.1-1.0 is reasonable) -->
+                  <friction>0.5</friction>  <!-- Static friction -->
+                </dynamics>
                 <command_interface name="position"/>
                 <state_interface name="position">
@@ -42,4 +69,5 @@
                 </state_interface>
                 <state_interface name="velocity"/>
+                <state_interface name="effort"/>
             </joint>
         </ros2_control>
